Commit message: wip

File: bluer_ugv/assets/arzhang4_description/urdf/arzhang4.urdf (robot description, URDF)
Before this commit: robot arzhang4, 5 links, 4 joints
Joints:
- joint wheel_fl_joint: origin xyz=0.19999999999999998 0.15000000000000002 0.1 rpy=0 0 0 -> xyz=0.2 0.15 0.1 rpy=0 0 0
- joint wheel_fr_joint: origin xyz=0.19999999999999998 -0.15000000000000002 0.1 rpy=0 0 0 -> xyz=0.2 -0.15 0.1 rpy=0 0 0
- joint wheel_rl_joint: origin xyz=-0.19999999999999998 0.15000000000000002 0.1 rpy=0 0 0 -> xyz=-0.2 0.15 0.1 rpy=0 0 0
- joint wheel_rr_joint: origin xyz=-0.19999999999999998 -0.15000000000000002 0.1 rpy=0 0 0 -> xyz=-0.2 -0.15 0.1 rpy=0 0 0

File: bluer_ugv/assets/arzhang4_description/urdf/arzhang4.urdf.xacro (robot description, xacro)
@@ -1,34 +1,35 @@
 <?xml version="1.0"?>
-<robot xmlns:xacro="http://www.ros.org/wiki/xacro" name="arzhang4">
+<robot name="arzhang4" xmlns:xacro="http://ros.org/wiki/xacro">
   <!-- ================= PARAMETERS ================= -->
-  <xacro:property name="chassis_length" value="0.60"/>
-  <xacro:property name="chassis_width"  value="0.40"/>
-  <xacro:property name="chassis_height" value="0.18"/>
-  <xacro:property name="wheel_radius" value="0.10"/>
-  <xacro:property name="wheel_width"  value="0.05"/>
-  <xacro:property name="wheel_separation" value="${chassis_width - 0.10}"/>
+  <xacro:property name="base_length" value="0.6" />
+  <xacro:property name="base_width" value="0.4" />
+  <xacro:property name="base_height" value="0.18" />
+  <xacro:property name="wheel_radius" value="0.1" />
+  <xacro:property name="wheel_width" value="0.05" />
+  <xacro:property name="wheel_x" value="0.2" />
+  <xacro:property name="wheel_y" value="0.15" />
+  <xacro:property name="wheel_z" value="0.1" />
   <!-- ================= BASE LINK ================= -->
   <link name="base_link">
     <inertial>
-      <origin xyz="0 0 ${chassis_height/2}" rpy="0 0 0"/>
-      <mass value="12.0"/>
-      <inertia
-        ixx="0.20" ixy="0.0" ixz="0.0"
+      <origin xyz="0 0 ${base_height/2}" rpy="0 0 0" />
+      <mass value="12.0" />
+      <inertia ixx="0.20" ixy="0.0" ixz="0.0"
         iyy="0.35" iyz="0.0"
-        izz="0.45"/>
+        izz="0.45" />
     </inertial>
     <visual>
-      <origin xyz="0 0 ${chassis_height/2}" rpy="0 0 0"/>
+      <origin xyz="0 0 ${base_height/2}" rpy="0 0 0" />
       <geometry>
-        <box size="${chassis_length} ${chassis_width} ${chassis_height}"/>
+        <box size="${base_length} ${base_width} ${base_height}" />
       </geometry>
       <material name="gray">
-        <color rgba="0.5 0.5 0.5 1.0"/>
+        <color rgba="0.6 0.6 0.6 1.0" />
       </material>
     </visual>
     <collision>
-      <origin xyz="0 0 ${chassis_height/2}" rpy="0 0 0"/>
+      <origin xyz="0 0 ${base_height/2}" rpy="0 0 0" />
       <geometry>
-        <box size="${chassis_length} ${chassis_width} ${chassis_height}"/>
+        <box size="${base_length} ${base_width} ${base_height}" />
       </geometry>
     </collision>
@@ -38,57 +39,50 @@
     <link name="${name}">
       <inertial>
-        <origin xyz="0 0 0" rpy="0 0 0"/>
-        <mass value="1.0"/>
-        <inertia
-          ixx="0.001" ixy="0.0" ixz="0.0"
+        <origin xyz="0 0 0" rpy="0 0 0" />
+        <mass value="1.0" />
+        <inertia ixx="0.001" ixy="0.0" ixz="0.0"
           iyy="0.001" iyz="0.0"
-          izz="0.001"/>
+          izz="0.001" />
       </inertial>
+      <!-- IMPORTANT: rotate cylinder so its Z-axis becomes Y (wheel axle) -->
       <visual>
-        <origin xyz="0 0 0" rpy="0 1.5708 0"/>
+        <origin xyz="0 0 0" rpy="1.5708 0 0" />
         <geometry>
-          <cylinder radius="${wheel_radius}" length="${wheel_width}"/>
+          <cylinder radius="${wheel_radius}" length="${wheel_width}" />
         </geometry>
         <material name="black">
-          <color rgba="0.1 0.1 0.1 1.0"/>
+          <color rgba="0.1 0.1 0.1 1.0" />
         </material>
       </visual>
       <collision>
-        <origin xyz="0 0 0" rpy="0 1.5708 0"/>
+        <origin xyz="0 0 0" rpy="1.5708 0 0" />
         <geometry>
-          <cylinder radius="${wheel_radius}" length="${wheel_width}"/>
+          <cylinder radius="${wheel_radius}" length="${wheel_width}" />
         </geometry>
       </collision>
     </link>
     <joint name="${name}_joint" type="continuous">
-      <parent link="base_link"/>
-      <child link="${name}"/>
-      <origin xyz="${x} ${y} ${wheel_radius}" rpy="0 0 0"/>
-      <axis xyz="0 1 0"/>
+      <parent link="base_link" />
+      <child link="${name}" />
+      <origin xyz="${x} ${y} ${wheel_z}" rpy="0 0 0" />
+      <!-- Axle along Y -->
+      <axis xyz="0 1 0" />
     </joint>
   </xacro:macro>
-  <!-- ================= 4 WHEELS ================= -->
-  <xacro:wheel name="wheel_fl"
-               x="${ chassis_length/2 - 0.10}"
-               y="${ wheel_separation/2}"/>
-  <xacro:wheel name="wheel_fr"
-               x="${ chassis_length/2 - 0.10}"
-               y="${-wheel_separation/2}"/>
-  <xacro:wheel name="wheel_rl"
-               x="${-chassis_length/2 + 0.10}"
-               y="${ wheel_separation/2}"/>
-  <xacro:wheel name="wheel_rr"
-               x="${-chassis_length/2 + 0.10}"
-               y="${-wheel_separation/2}"/>
-  <!-- ================= GAZEBO SIM DIFF DRIVE ================= -->
+  <!-- ================= FOUR WHEELS ================= -->
+  <xacro:wheel name="wheel_fl" x="${ wheel_x}" y="${ wheel_y}" />
+  <xacro:wheel name="wheel_fr" x="${ wheel_x}" y="${-wheel_y}" />
+  <xacro:wheel name="wheel_rl" x="${-wheel_x}" y="${ wheel_y}" />
+  <xacro:wheel name="wheel_rr" x="${-wheel_x}" y="${-wheel_y}" />
+  <!-- ================= GAZEBO DIFF DRIVE ================= -->
   <gazebo>
     <plugin filename="gz-sim-diff-drive-system"
-            name="gz::sim::systems::DiffDrive">
+      name="gz::sim::systems::DiffDrive">
       <left_joint>wheel_fl_joint</left_joint>
       <left_joint>wheel_rl_joint</left_joint>
       <right_joint>wheel_fr_joint</right_joint>
       <right_joint>wheel_rr_joint</right_joint>
-      <wheel_separation>${wheel_separation}</wheel_separation>
-      <wheel_radius>${wheel_radius}</wheel_radius>
+      <wheel_separation>0.3</wheel_separation>
+      <wheel_radius>0.1</wheel_radius>
       <topic>cmd_vel</topic>
       <odom_topic>odom</odom_topic>

Commit message: wip

File: bluer_ugv/assets/arzhang4_description/urdf/arzhang4.urdf (robot description, URDF)
Before this commit: robot arzhang4, 5 links, 4 joints
Links:
- link base_link: geometry collision box size=0.6 0.26 0.12; visual box size=0.6 0.26 0.12
- link wheel_fl: geometry collision cylinder length=0.1 radius=0.13; visual cylinder length=0.1 radius=0.13
- link wheel_fr: geometry collision cylinder length=0.1 radius=0.13; visual cylinder length=0.1 radius=0.13
- link wheel_rl: geometry collision cylinder length=0.1 radius=0.13; visual cylinder length=0.1 radius=0.13
- link wheel_rr: geometry collision cylinder length=0.1 radius=0.13; visual cylinder length=0.1 radius=0.13
Joints:
- joint wheel_fl_joint: origin xyz=0.2 0.15 0.1 rpy=0 0 0 -> xyz=0.2 0.15 0.13 rpy=0 0 0
- joint wheel_fr_joint: origin xyz=0.2 -0.15 0.1 rpy=0 0 0 -> xyz=0.2 -0.15 0.13 rpy=0 0 0
- joint wheel_rl_joint: origin xyz=-0.2 0.15 0.1 rpy=0 0 0 -> xyz=-0.2 0.15 0.13 rpy=0 0 0
- joint wheel_rr_joint: origin xyz=-0.2 -0.15 0.1 rpy=0 0 0 -> xyz=-0.2 -0.15 0.13 rpy=0 0 0

File: bluer_ugv/assets/arzhang4_description/urdf/arzhang4.urdf.xacro (robot description, xacro)
@@ -3,11 +3,11 @@
   <!-- ================= PARAMETERS ================= -->
   <xacro:property name="base_length" value="0.6" />
-  <xacro:property name="base_width" value="0.4" />
-  <xacro:property name="base_height" value="0.18" />
-  <xacro:property name="wheel_radius" value="0.1" />
-  <xacro:property name="wheel_width" value="0.05" />
+  <xacro:property name="base_width" value="0.26" />
+  <xacro:property name="base_height" value="0.12" />
+  <xacro:property name="wheel_radius" value="0.13" />
+  <xacro:property name="wheel_width" value="0.1" />
   <xacro:property name="wheel_x" value="0.2" />
   <xacro:property name="wheel_y" value="0.15" />
-  <xacro:property name="wheel_z" value="0.1" />
+  <xacro:property name="wheel_z" value="0.13" />
   <!-- ================= BASE LINK ================= -->
   <link name="base_link">

Commit message: wip

File: bluer_ugv/assets/arzhang4_description/urdf/arzhang4.urdf (robot description, URDF)
Before this commit: robot arzhang4, 5 links, 4 joints
Joints:
- joint wheel_fl_joint: origin xyz=0.2 0.15 0.13 rpy=0 0 0 -> xyz=0.2 0.15 0.06 rpy=0 0 0
- joint wheel_fr_joint: origin xyz=0.2 -0.15 0.13 rpy=0 0 0 -> xyz=0.2 -0.15 0.06 rpy=0 0 0
- joint wheel_rl_joint: origin xyz=-0.2 0.15 0.13 rpy=0 0 0 -> xyz=-0.2 0.15 0.06 rpy=0 0 0
- joint wheel_rr_joint: origin xyz=-0.2 -0.15 0.13 rpy=0 0 0 -> xyz=-0.2 -0.15 0.06 rpy=0 0 0

File: bluer_ugv/assets/arzhang4_description/urdf/arzhang4.urdf.xacro (robot description, xacro)
@@ -9,5 +9,5 @@
   <xacro:property name="wheel_x" value="0.2" />
   <xacro:property name="wheel_y" value="0.15" />
-  <xacro:property name="wheel_z" value="0.13" />
+  <xacro:property name="wheel_z" value="0.06" />
   <!-- ================= BASE LINK ================= -->
   <link name="base_link">
